File: hardware/audio.kicad_sch (KiCad schematic)
At the start: 50 parts, among them J6 PJ-342, J7 4.4mm balanced, U14 SN74AVC4T774PWR, U15 PCA9306DCUR, U16 74LVC1G04, U17 CS43131-CNZR, U18 CS43131-CNZR, Y1 22.5792MHz, Y2 24.576MHz

Commit message: Use the chosen parts in the schematic, with their LCSC numbers
The headphone jacks are now real parts. The 3.5 mm SHOU HAN PJ-342 is a
3-pole stereo jack, per its drawing: tip 3, ring 6, sleeve 5 and 2, and a
switch on tip and ring that touches them while no plug is in. Its tip
switch drives the left DAC's HP_DETECT, so the firmware sets
HPDETECT_INV. The 4.4 mm jack is the Kinghelm KH-PJ-44002-12DBAP-A: two
pins per pole in Pentaconn order and a separate plug switch from DET_44
to ground.

Checked against the datasheets: the oscillators' OE is high or open =
running and tri-state when low, so they can share MCLK; the GL823K's VDD
and VDDA are both its own 3.3 V. The CS43131 FILT capacitors are 22 uF
0805 25 V now, about 15-19 uF under bias where a 15 uF part would keep
about 11. The e-paper circuit follows the GDEY037T03-T02 reference: VPP
(pin 19) left open and a 1 MOhm gate pull-down, R1 and R2 in 0603.

Every assembled part has an LCSC number: the passives are in a table
checked on lcsc.com. 49.9k had no stock, so the TPS2553 limit resistor is
47k (about 0.5 A). The touch and microSD footprints are the real ones.
Parts:
- removed C79: 2.2uF, Capacitor_SMD:C_0603_1608Metric, symbol Device:C
- removed J6: PJ-342, dap:Jack_3.5mm_PJ-342_standin, symbol dap:AudioJack_3.5_TRRS
- removed J7: 4.4mm balanced, dap:Jack_4.4mm_standin, symbol dap:AudioJack_4.4
- added C45: 100nF, Capacitor_SMD:C_0402_1005Metric, symbol Device:C
- added J6: PJ-342, dap:Jack_3.5mm_PJ-342, symbol dap:PJ-342
- added J7: KH-PJ-44002-12DBAP-A, dap:Jack_4.4mm_KH-PJ-44002-12DBAP-A, symbol dap:KH-PJ-44002
- C46, C47, C48, C49, C50, C51, C52, C53, C66, C67: LCSC (none) -> C1525
- C54, C68: value 100nF -> 4.7uF; footprint Capacitor_SMD:C_0402_1005Metric -> Capacitor_SMD:C_0603_1608Metric; LCSC (none) -> C19666
- C55, C69: value 4.7uF -> 2.2uF; LCSC (none) -> C23630
- C56, C70: value 2.2uF -> 22uF; footprint Capacitor_SMD:C_0603_1608Metric -> Capacitor_SMD:C_0805_2012Metric; LCSC (none) -> C45783
- C57, C71: value 15uF -> 22uF; LCSC (none) -> C45783
- C58, C72: value 15uF -> 2.2uF; footprint Capacitor_SMD:C_0805_2012Metric -> Capacitor_SMD:C_0603_1608Metric; LCSC (none) -> C23630
- C59, C60, C61, C62, C63, C64, C73, C74, C75, C76, C77, C78: LCSC (none) -> C23630
- C65: value 2.2uF -> 100nF; footprint Capacitor_SMD:C_0603_1608Metric -> Capacitor_SMD:C_0402_1005Metric; LCSC (none) -> C1525
- R31: LCSC (none) -> C25764
- R32, R33: LCSC (none) -> C25900
- R34, R35: LCSC (none) -> C25092
- R36: LCSC (none) -> C25903
Connections:
- net +3V3: now also C45.1; no longer C46.1
- net 1V8_A: now also C55.1, C56.2, C69.1, C70.2; no longer C56.1, C57.2, C70.1, C71.2
- net 1V8_CP: now also C60.1, C74.1; no longer C61.1, C75.1
- net 1V8_D: now also C46.1, C48.1, C65.1; no longer C47.1, C53.1, C67.1
- net DACL_FILTN: now also C57.1; no longer C58.1
- net DACL_FILTP: now also C56.1; no longer C57.1
- net DACL_FLYC_VCP: now also C63.2, C64.1; no longer C64.2, C65.1
- net DACL_FLYN_VA: now also C59.2; no longer C60.2
- net DACL_FLYN_VCP: now also C64.2; no longer C65.2
- net DACL_FLYP_VA: now also C59.1; no longer C60.1
- net DACL_FLYP_VCP: now also C63.1; no longer C64.1
- net DACL_NVA: now also C57.2, C58.1; no longer C58.2, C59.1
- net DACL_VCPF_N: now also C62.1; no longer C63.1
- net DACL_VCPF_P: now also C61.1; no longer C62.1
- net DACR_FILTN: now also C71.1; no longer C72.1
- net DACR_FILTP: now also C70.1; no longer C71.1
- net DACR_FLYC_VCP: now also C77.2, C78.1; no longer C78.2
- net DACR_FLYN_VA: now also C73.2; no longer C74.2
- net DACR_FLYN_VCP: now also C78.2
- net DACR_FLYP_VA: now also C73.1; no longer C74.1
- net DACR_FLYP_VCP: now also C77.1; no longer C78.1
- net DACR_NVA: now also C71.2, C72.1; no longer C72.2, C73.1
- net DACR_VCPF_N: now also C76.1; no longer C77.1
- net DACR_VCPF_P: now also C75.1; no longer C76.1
- net DET_35: now also J6.4 (TSW)
- net DET_44: now also J7.11 (SW_A)
- net GND: now also C58.2, C60.2, C65.2, C72.2, C74.2, C45.2, J7.12 (SW_B); no longer C56.2, C59.2, C63.2, C70.2, C73.2, C77.2
- net HP_GND: now also J6.2 (S), J6.5 (S), J7.1 (S), J7.6 (S)
- net I2C_VREF2: now also C47.1; no longer C48.1
- net OUT_LN: now also J7.4 (L-), J7.9 (L-)
- net OUT_LP: now also J6.3 (T), J7.10 (L+), J7.5 (L+)
- net OUT_RN: now also J7.2 (R-), J7.7 (R-)
- net OUT_RP: now also J6.6 (R), J7.3 (R+), J7.8 (R+)
- net VP: now also C53.1, C67.1; no longer C55.1, C69.1
- no-connect marks 18 -> 19
Other:
- note added: "3.5 mm takes L+ and R+ only. HP_GND joins GND at the jacks"
- note added: "Headphone jacks, both on the back of the board: they share the outputs;"
- note removed: "Headphone jacks: both share the outputs; 3.5 mm takes L+ and R+"
- note removed: "only. HP_GND joins GND at the jacks"
