File: hardware/display.kicad_sch (KiCad schematic)
At the start: 24 parts, among them J2 E-paper FPC, J3 Touch FPC, Q1 Si1308EDL

Commit message: Use the chosen parts in the schematic, with their LCSC numbers
The headphone jacks are now real parts. The 3.5 mm SHOU HAN PJ-342 is a
3-pole stereo jack, per its drawing: tip 3, ring 6, sleeve 5 and 2, and a
switch on tip and ring that touches them while no plug is in. Its tip
switch drives the left DAC's HP_DETECT, so the firmware sets
HPDETECT_INV. The 4.4 mm jack is the Kinghelm KH-PJ-44002-12DBAP-A: two
pins per pole in Pentaconn order and a separate plug switch from DET_44
to ground.

Checked against the datasheets: the oscillators' OE is high or open =
running and tri-state when low, so they can share MCLK; the GL823K's VDD
and VDDA are both its own 3.3 V. The CS43131 FILT capacitors are 22 uF
0805 25 V now, about 15-19 uF under bias where a 15 uF part would keep
about 11. The e-paper circuit follows the GDEY037T03-T02 reference: VPP
(pin 19) left open and a 1 MOhm gate pull-down, R1 and R2 in 0603.

Every assembled part has an LCSC number: the passives are in a table
checked on lcsc.com. 49.9k had no stock, so the TPS2553 limit resistor is
47k (about 0.5 A). The touch and microSD footprints are the real ones.
Parts:
- removed C35: 1uF, Capacitor_SMD:C_0402_1005Metric, symbol Device:C
- C23, C24: LCSC (none) -> C98192
- C25, C26, C27, C28, C29, C30, C31, C32, C33: LCSC (none) -> C15849
- C34: value 1uF/50V -> 1uF; footprint Capacitor_SMD:C_0603_1608Metric -> Capacitor_SMD:C_0402_1005Metric; LCSC (none) -> C52923
- J2: Note pin 1 NC, 6/7 temperature sensor I2C unused -> pin 1 NC, 6/7 temperature sensor I2C unused, 19 VPP (test p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
- J3: footprint Connector_FFC-FPC:Hirose_FH12-6S-0.5SH_1x06-1MP_P0.50mm_Horizontal -> Connector_FFC-FPC:Jushuo_AFC07-S06FCA-00_1x6-1MP_P0.50_Horizontal; Note footprint stands in for the Jushuo AFC07-S06FCA-00 until st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 -> bottom contact, like the e-paper connector; the 56 mm touch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
- L3: LCSC (none) -> C354566
- R21: value 10k -> 1M; footprint Resistor_SMD:R_0402_1005Metric -> Resistor_SMD:R_0603_1608Metric; LCSC (none) -> C22935
- R22: footprint Resistor_SMD:R_0402_1005Metric -> Resistor_SMD:R_0603_1608Metric; LCSC (none) -> C23411
- R23, R24: LCSC (none) -> C25744
Connections:
- net +3V3: now also C34.1
- net EPD_PREVGH: now also C30.1; no longer C31.1
- net EPD_PREVGL: now also C32.1; no longer C33.1
- net EPD_VCOM: now also C33.1; no longer C34.1
- net EPD_VSH: now also C29.1; no longer C30.1
- net EPD_VSL: now also C31.1; no longer C32.1
- net EPD_VPP: no longer names the net of J2.19 (Pin_19)
- net EPD_VPP: no longer C29.1
- no-connect marks 3 -> 4
Other:
- note added: "E-paper GDEY037T03 (UC8253), 24-pin FPC: the reference circuit in the GDEY037T03-T02"
- note added: "spec (p. 35), 0.47 R sense for UC driver ICs. BS1 low = 4-wire SPI"
- note removed: "E-paper GDEY037T03 (UC8253), 24-pin FPC: Good Display's reference booster circuit, 0.47"
- note removed: "R sense for UC driver ICs. BS1 low = 4-wire SPI"
