File: hardware/mcu.kicad_sch (KiCad schematic)
At the start: 26 parts, among them SW1 Play, SW2 Power, SW3 Vol+, SW4 Vol-, U8 ESP32-S3-WROOM-1-N16R8

Commit message: Use the chosen parts in the schematic, with their LCSC numbers
The headphone jacks are now real parts. The 3.5 mm SHOU HAN PJ-342 is a
3-pole stereo jack, per its drawing: tip 3, ring 6, sleeve 5 and 2, and a
switch on tip and ring that touches them while no plug is in. Its tip
switch drives the left DAC's HP_DETECT, so the firmware sets
HPDETECT_INV. The 4.4 mm jack is the Kinghelm KH-PJ-44002-12DBAP-A: two
pins per pole in Pentaconn order and a separate plug switch from DET_44
to ground.

Checked against the datasheets: the oscillators' OE is high or open =
running and tri-state when low, so they can share MCLK; the GL823K's VDD
and VDDA are both its own 3.3 V. The CS43131 FILT capacitors are 22 uF
0805 25 V now, about 15-19 uF under bias where a 15 uF part would keep
about 11. The e-paper circuit follows the GDEY037T03-T02 reference: VPP
(pin 19) left open and a 1 MOhm gate pull-down, R1 and R2 in 0603.

Every assembled part has an LCSC number: the passives are in a table
checked on lcsc.com. 49.9k had no stock, so the TPS2553 limit resistor is
47k (about 0.5 A). The touch and microSD footprints are the real ones.
Parts:
- C19: LCSC (none) -> C15850
- C20, C22: LCSC (none) -> C1525
- C21: LCSC (none) -> C52923
- D1: LCSC (none) -> C72043
- R10, R11, R13, R14, R15, R8, R9: LCSC (none) -> C25741
- R12, R7: LCSC (none) -> C25744
- R16, R17: LCSC (none) -> C26083
- R18, R19: LCSC (none) -> C25900
- R20: LCSC (none) -> C11702
