File: hardware/usb_storage.kicad_sch (KiCad schematic)
At the start: 23 parts, among them J4 USB-C, J5 microSD, U10 TUSB320LIRWBR, U11 FSUSB42MUX, U12 GL823K-HCY04, U13 TS3A27518EPWR, U9 USBLC6-2SC6

Commit message: Use the chosen parts in the schematic, with their LCSC numbers
The headphone jacks are now real parts. The 3.5 mm SHOU HAN PJ-342 is a
3-pole stereo jack, per its drawing: tip 3, ring 6, sleeve 5 and 2, and a
switch on tip and ring that touches them while no plug is in. Its tip
switch drives the left DAC's HP_DETECT, so the firmware sets
HPDETECT_INV. The 4.4 mm jack is the Kinghelm KH-PJ-44002-12DBAP-A: two
pins per pole in Pentaconn order and a separate plug switch from DET_44
to ground.

Checked against the datasheets: the oscillators' OE is high or open =
running and tri-state when low, so they can share MCLK; the GL823K's VDD
and VDDA are both its own 3.3 V. The CS43131 FILT capacitors are 22 uF
0805 25 V now, about 15-19 uF under bias where a 15 uF part would keep
about 11. The e-paper circuit follows the GDEY037T03-T02 reference: VPP
(pin 19) left open and a 1 MOhm gate pull-down, R1 and R2 in 0603.

Every assembled part has an LCSC number: the passives are in a table
checked on lcsc.com. 49.9k had no stock, so the TPS2553 limit resistor is
47k (about 0.5 A). The touch and microSD footprints are the real ones.
Parts:
- removed C45: 100nF, Capacitor_SMD:C_0402_1005Metric, symbol Device:C
- added C35: 10uF, Capacitor_SMD:C_0805_2012Metric, symbol Device:C
- C36, C44: value 10uF -> 100nF; footprint Capacitor_SMD:C_0805_2012Metric -> Capacitor_SMD:C_0402_1005Metric; LCSC (none) -> C1525
- C37, C38, C42: LCSC (none) -> C1525
- C39: value 100nF -> 4.7uF; footprint Capacitor_SMD:C_0402_1005Metric -> Capacitor_SMD:C_0603_1608Metric; LCSC (none) -> C19666
- C40: value 4.7uF -> 1uF; footprint Capacitor_SMD:C_0603_1608Metric -> Capacitor_SMD:C_0402_1005Metric; LCSC (none) -> C52923
- C41: value 1uF -> 100nF; LCSC (none) -> C1525
- C43: value 100nF -> 10uF; footprint Capacitor_SMD:C_0402_1005Metric -> Capacitor_SMD:C_0805_2012Metric; LCSC (none) -> C15850
- J5: footprint Connector_Card:microSD_HC_Hirose_DM3D-SF -> dap:microSD_TF-01A; Note footprint stands in for the TF-01A until stage 3 -> Hroparts TF-01A push-push socket; its card-detect contact (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
- R25: LCSC (none) -> C423127
- R26, R27, R28, R29, R30: LCSC (none) -> C25744
Connections:
- net +3V3: now also C37.1, C42.1; no longer C39.1
- net GL_3V3: now also C40.1; no longer C42.1
- net GND: now also C35.2
- net VBUS: now also C39.1, C35.1; no longer C37.1, C40.1
